Commit message: camera frames

File: urdf/reachy.URDF.xacro (robot description, xacro)
@@ -103,5 +103,5 @@
     </visual>
     <collision>
-        <origin xyz="-0.009 -0.002 0.059" rpy="1.57 0.0 0.0"/>
+        <origin xyz="-0.009 -0.002 0.059" rpy="${pi/2.0} 0.0 0.0"/>
         <geometry>
             <cylinder length="0.15" radius="0.06" />
@@ -156,10 +156,10 @@
 <link name="r_shoulder">
     <inertial>
-        <origin xyz="-0.016 0.036 0.0" rpy="1.57 1.57 0.0"/>
+        <origin xyz="-0.016 0.036 0.0" rpy="${pi/2.0} ${pi/2.0} 0.0"/>
         <mass value="0.053"/>
         <inertia ixx="3.308e-4" ixy="9.972e-8" ixz="-2.037e-9" iyy="4.650e-5" iyz="2.113e-6" izz="3.545e-5"/>
     </inertial>
     <visual name="">
-        <origin xyz="0.0 0.04 0.0" rpy="1.57 1.57 0.0"/>
+        <origin xyz="0.0 0.04 0.0" rpy="${pi/2.0} ${pi/2.0} 0.0"/>
         <geometry>
             <mesh filename="file://$(find reachy_description)/meshes/shoulder.dae"/>
@@ -167,5 +167,5 @@
     </visual>
     <collision>
-        <origin xyz="0.0 0.04 0.0" rpy="1.57 1.57 0.0"/>
+        <origin xyz="0.0 0.04 0.0" rpy="${pi/2.0} ${pi/2.0} 0.0"/>
         <geometry>
             <cylinder length="0.09" radius="0.035" />
@@ -271,5 +271,5 @@
     <inertial>
         <!-- <origin xyz="0.032 -0.008 0.0" rpy="0.0 1.57 0.0"/> -->
-        <origin xyz="0.0 -0.008 0.0" rpy="0.0 1.57 0.0"/>
+        <origin xyz="0.0 -0.008 0.0" rpy="0.0 ${pi/2.0} 0.0"/>
         <mass value="0.173"/>
         <!-- <inertia ixx="1.083e-4" ixy="-3.476e-5" ixz="1.331e-6" iyy="1.421e-4" iyz="6.730e-7" izz="2.112e-4"/> -->
@@ -277,5 +277,5 @@
     </inertial>
     <visual name="">
-        <origin xyz="0.0 0.0 0.0" rpy="0.0 1.57 0.0"/>
+        <origin xyz="0.0 0.0 0.0" rpy="0.0 ${pi/2.0} 0.0"/>
         <geometry>
             <mesh filename="file://$(find reachy_description)/meshes/r_gripper_thumb.dae"/>
@@ -283,5 +283,5 @@
     </visual>
     <collision>
-        <origin xyz="0.0 0.02 -0.06" rpy="0.0 1.57 0.0"/>
+        <origin xyz="0.0 0.02 -0.06" rpy="0.0 ${pi/2.0} 0.0"/>
         <geometry>
             <box size="0.1 0.012 0.035" />
@@ -292,5 +292,5 @@
     <inertial>
         <!-- <origin xyz="-0.005 -0.043 -0.0" rpy="0.0 1.57 0.0"/> -->
-        <origin xyz="-0.00 -0.005 -0.0" rpy="1.57 0.0 1.57"/>
+        <origin xyz="-0.00 -0.005 -0.0" rpy="${pi/2.0} 0.0 ${pi/2.0}"/>
         <mass value="0.035"/>
         <!-- <inertia ixx="9.166e-5" ixy="-6.559e-6" ixz="-3.952e-8" iyy="1.062e-5" iyz="5.276e-9" izz="8.704e-5"/> -->
@@ -298,5 +298,5 @@
     </inertial>
     <visual name="">
-        <origin xyz="0.0 0.0 0.0" rpy="0.0 1.57 0.0"/>
+        <origin xyz="0.0 0.0 0.0" rpy="0.0 ${pi/2.0} 0.0"/>
         <geometry>
             <mesh filename="file://$(find reachy_description)/meshes/r_gripper_finger.dae"/>
@@ -304,5 +304,5 @@
     </visual>
     <collision>
-        <origin xyz="0.0 -0.01 -0.02" rpy="0.0 1.57 0.0"/>
+        <origin xyz="0.0 -0.01 -0.02" rpy="0.0 ${pi/2.0} 0.0"/>
         <geometry>
             <box size="0.1 0.012 0.035" />
@@ -316,10 +316,10 @@
 <link name="l_shoulder">
     <inertial>
-        <origin xyz="-0.016 -0.036 0.0" rpy="-1.57 1.57 0.0"/>
+        <origin xyz="-0.016 -0.036 0.0" rpy="${-pi/2.0} ${pi/2.0} 0.0"/>
         <mass value="0.053"/>
         <inertia ixx="3.308e-4" ixy="9.972e-8" ixz="-2.037e-9" iyy="4.650e-5" iyz="2.113e-6" izz="3.545e-5"/>
     </inertial>
     <visual name="">
-        <origin xyz="0.0 -0.04 0.0" rpy="-1.57 1.57 0.0"/>
+        <origin xyz="0.0 -0.04 0.0" rpy="${-pi/2.0} ${pi/2.0} 0.0"/>
         <geometry>
             <mesh filename="file://$(find reachy_description)/meshes/shoulder.dae"/>
@@ -327,5 +327,5 @@
     </visual>
     <collision>
-        <origin xyz="0.0 -0.04 0.0" rpy="-1.57 1.57 0.0"/>
+        <origin xyz="0.0 -0.04 0.0" rpy="${-pi/2.0} ${pi/2.0} 0.0"/>
         <geometry>
             <cylinder length="0.09" radius="0.035" />
@@ -431,5 +431,5 @@
     <inertial>
         <!-- <origin xyz="0.032 0.008 0.0" rpy="0.0 1.57 0.0"/> -->
-        <origin xyz="0.0 0.008 0.0" rpy="0.0 1.57 0.0"/>
+        <origin xyz="0.0 0.008 0.0" rpy="0.0 ${pi/2.0} 0.0"/>
         <mass value="0.173"/>
         <!-- <inertia ixx="1.088e+5" ixy="3.479e+4" ixz="1.357e+3" iyy="1.422e+5" iyz="-7.930e+2" izz="2.116e+5"/> -->
@@ -437,5 +437,5 @@
     </inertial>
     <visual name="">
-        <origin xyz="0.0 0.0 0.0" rpy="0.0 1.57 0.0"/>
+        <origin xyz="0.0 0.0 0.0" rpy="0.0 ${pi/2.0} 0.0"/>
         <geometry>
             <mesh filename="file://$(find reachy_description)/meshes/l_gripper_thumb.dae"/>
@@ -443,5 +443,5 @@
     </visual>
     <collision>
-        <origin xyz="0.0 -0.02 -0.06" rpy="0.0 1.57 0.0"/>
+        <origin xyz="0.0 -0.02 -0.06" rpy="0.0 ${pi/2.0} 0.0"/>
         <geometry>
             <box size="0.1 0.012 0.035" />
@@ -452,5 +452,5 @@
     <inertial>
         <!-- <origin xyz="0.005 -0.043 0.0" rpy="0.0 1.57 0.0"/> -->
-        <origin xyz="-0.00 0.005 -0.0" rpy="1.57 0.0 1.57"/>
+        <origin xyz="-0.00 0.005 -0.0" rpy="${pi/2.0} 0.0 ${pi/2.0}"/>
         <mass value="0.035"/>
         <!-- <inertia ixx="9.165e-5" ixy="6.559e-6" ixz="3.609e-10" iyy="1.062e-5" iyz="4.666e-9" izz="8.705e-5"/> -->
@@ -458,5 +458,5 @@
     </inertial>
     <visual name="">
-        <origin xyz="0.0 0.0 0.0" rpy="0.0 1.57 0.0"/>
+        <origin xyz="0.0 0.0 0.0" rpy="0.0 ${pi/2.0} 0.0"/>
         <geometry>
             <mesh filename="file://$(find reachy_description)/meshes/l_gripper_finger.dae"/>
@@ -464,5 +464,5 @@
     </visual>
     <collision>
-        <origin xyz="0.0 0.01 -0.02" rpy="0.0 1.57 0.0"/>
+        <origin xyz="0.0 0.01 -0.02" rpy="0.0 ${pi/2.0} 0.0"/>
         <geometry>
             <box size="0.1 0.012 0.035" />
@@ -508,5 +508,5 @@
     <child link="r_shoulder"/>
     <axis xyz="0 1 0"/>
-   <limit lower="-2.618" upper="1.57" effort="10." velocity="0.0"/>
+   <limit lower="-2.618" upper="${pi/2.0}" effort="10." velocity="0.0"/>
     <dynamics damping="${damping}" friction="${friction}" />
 </joint>
@@ -516,5 +516,5 @@
     <child link="r_shoulder_x"/>
     <axis xyz="1 0 0"/>
-   <limit lower="-3.14" upper="0.174" effort="10." velocity="0.0"/>
+   <limit lower="${-pi}" upper="0.174" effort="10." velocity="0.0"/>
     <dynamics damping="${damping}" friction="${friction}" />
 </joint>
@@ -524,5 +524,5 @@
     <child link="r_upper_arm"/>
     <axis xyz="0 0 1"/>
-   <limit lower="-1.57" upper="1.57" effort="10." velocity="0.0"/>
+   <limit lower="${-pi/2.0}" upper="${pi/2.0}" effort="10." velocity="0.0"/>
     <dynamics damping="${damping}" friction="${friction}" />
 </joint>
@@ -577,5 +577,5 @@
         <ros>
           <!-- Add namespace and remap the default topic -->
-          <namespace>/force_sensors</namespace>
+          <namespace>/right_force_sensor</namespace>
           <argument>wrench:=r_gripper_ft_sensor</argument>
         </ros>
@@ -600,5 +600,5 @@
     <child link="l_shoulder"/>
     <axis xyz="0 1 0"/>
-   <limit lower="-2.618" upper="1.57" effort="10." velocity="0.0"/>
+   <limit lower="-2.618" upper="${pi/2.0}" effort="10." velocity="0.0"/>
     <dynamics damping="${damping}" friction="${friction}" />
 </joint>
@@ -608,5 +608,5 @@
     <child link="l_shoulder_x"/>
     <axis xyz="1 0 0"/>
-   <limit lower="-0.174" upper="3.14" effort="10." velocity="0.0"/>
+   <limit lower="-0.174" upper="${pi}" effort="10." velocity="0.0"/>
     <dynamics damping="${damping}" friction="${friction}" />
 </joint>
@@ -616,5 +616,5 @@
     <child link="l_upper_arm"/>
     <axis xyz="0 0 1"/>
-   <limit lower="-1.57" upper="1.57" effort="10." velocity="0.0"/>
+   <limit lower="${-pi/2.0}" upper="${pi/2.0}" effort="10." velocity="0.0"/>
     <dynamics damping="${damping}" friction="${friction}" />
 </joint>
@@ -666,5 +666,5 @@
         <ros>
           <!-- Add namespace and remap the default topic -->
-          <namespace>/force_sensors</namespace>
+          <namespace>/left_force_sensor</namespace>
           <argument>wrench:=l_gripper_ft_sensor</argument>
         </ros>
@@ -794,5 +794,5 @@
 <link name="bottom_neck_arm">
     <visual name="">
-        <origin xyz="0.0 0.0 0.0" rpy="0.0 0.0 -1.57"/>
+        <origin xyz="0.0 0.0 0.0" rpy="0.0 0.0 ${-pi/2.0}"/>
         <geometry>
             <mesh filename="file://$(find reachy_description)/meshes/orbita_arm.dae"/>
@@ -840,5 +840,5 @@
         image won't be aligned properly with the frame it is supposedly
         originating from -->
-    <origin xyz="0 0 0" rpy="0 0 0"/>
+    <origin xyz="0 0 0" rpy="${-pi/2.0} 0 ${-pi/2.0}"/>
     <parent link="left_camera"/>
     <child link="left_camera_optical"/>
@@ -875,5 +875,5 @@
         image won't be aligned properly with the frame it is supposedly
         originating from -->
-    <origin xyz="0 0 0" rpy="0 0 0"/>
+    <origin xyz="0 0 0" rpy="${-pi/2.0} 0 ${-pi/2.0}"/>
     <parent link="right_camera"/>
     <child link="right_camera_optical"/>
@@ -948,5 +948,5 @@
           </camera>
           <!-- Use camera, not camera_triggered -->
-          <plugin name="camera_controller" filename="libgazebo_ros_camera.so">
+          <plugin name="left_camera_controller" filename="libgazebo_ros_camera.so">
             <!-- <ros> -->
             <!--   <namespace>custom_ns</namespace> -->
@@ -991,5 +991,5 @@
           </camera>
           <!-- Use camera, not camera_triggered -->
-          <plugin name="camera_controller" filename="libgazebo_ros_camera.so">
+          <plugin name="right_camera_controller" filename="libgazebo_ros_camera.so">
             <!-- <ros> -->
             <!--   <namespace>custom_ns</namespace> -->
@@ -1037,5 +1037,5 @@
         image won't be aligned properly with the frame it is supposedly
         originating from -->
-    <origin xyz="0 0 0" rpy="0 0 0"/>
+    <origin xyz="0 0 0" rpy="${-pi/2.0} 0 ${-pi/2.0}"/>
     <parent link="depth_camera_link"/>
     <child link="depth_camera_optical"/>
