Commit message: fix antenna names

File: urdf/reachy.URDF (robot description, URDF)
Before this commit: robot reachy, 31 links, 30 joints
Links:
- removed link l_antenna
- removed link r_antenna
- added link l_antenna_link, mass 0.004; collision cylinder length=0.0 radius=0.0; visual mesh filename=package://reachy_description_ros2/meshes/antenna.dae
- added link r_antenna_link, mass 0.004; collision cylinder length=0.0 radius=0.0; visual mesh filename=package://reachy_description_ros2/meshes/antenna.dae
Joints:
- joint l_antenna: child l_antenna -> l_antenna_link
- joint r_antenna: child r_antenna -> r_antenna_link

File: urdf/reachy.URDF.xacro (robot description, xacro)
@@ -69,5 +69,5 @@
 </link>
 <link name="head_tip"/>
-<link name="l_antenna">
+<link name="l_antenna_link">
     <inertial>
         <origin xyz="-0.001 0.0 0.008" rpy="0.0 0.0 0.0"/>
@@ -88,5 +88,5 @@
     </collision>
 </link>
-<link name="r_antenna">
+<link name="r_antenna_link">
     <inertial>
         <origin xyz="-0.001 0.0 0.008" rpy="0.0 0.0 0.0"/>
@@ -435,5 +435,5 @@
     <origin xyz="-0.052 -0.057 0.086" rpy="-0.166 -1.054 1.11"/>
     <parent link="head"/>
-    <child link="r_antenna"/>
+    <child link="r_antenna_link"/>
     <axis xyz="0 0 1"/>
    <limit lower="-2.618" upper="2.618" effort="10." velocity="0.0"/>
@@ -442,5 +442,5 @@
     <origin xyz="-0.052 0.057 0.086" rpy="0.166 -1.054 -1.11"/>
     <parent link="head"/>
-    <child link="l_antenna"/>
+    <child link="l_antenna_link"/>
     <axis xyz="0 0 1"/>
    <limit lower="-2.618" upper="2.618" effort="10." velocity="0.0"/>

Commit message: gazebo working

File: urdf/reachy.URDF (robot description, URDF)
Before this commit: robot reachy, 31 links, 30 joints
Joints:
- removed joint l_antenna
- removed joint r_antenna
- added joint l_antenna_joint: type revolute, parent head, child l_antenna, origin xyz=-0.052 0.057 0.086 rpy=0.166 -1.054 -1.11, axis 0 0 1, limit lower=-2.618 upper=2.618 effort=10. velocity=0.0
- added joint r_antenna_joint: type revolute, parent head, child r_antenna, origin xyz=-0.052 -0.057 0.086 rpy=-0.166 -1.054 1.11, axis 0 0 1, limit lower=-2.618 upper=2.618 effort=10. velocity=0.0

File: urdf/reachy.URDF.xacro (robot description, xacro)
@@ -4,4 +4,17 @@
 <xacro:arg name="left_arm" default="true"/>
 <xacro:arg name="right_arm" default="true"/>
+<!-- pretty important for stability -->
+<xacro:property name="damping" value="0" />
+<xacro:property name="friction" value="0.1" />
+<xacro:macro name="xmass" params="value"><mass value="${value}" /></xacro:macro>
+<xacro:macro name="inertial_cuboid" params="mass xyz rpy x_length y_length z_length">
+  <inertial>
+    <xacro:xmass value="${mass}" />
+    <origin rpy="${rpy}" xyz="${xyz}"/>
+    <inertia ixx="${mass * (y_length*y_length + z_length*z_length) / 12}" ixy="0.0" ixz="0.0"
+             iyy="${mass * (x_length*x_length + z_length*z_length) / 12}" iyz="0.0"
+             izz="${mass * (x_length*x_length + y_length*y_length) / 12}" />
+  </inertial>
+</xacro:macro>
 <!-- Torso Link -->
   <material name="Grey">
@@ -28,4 +41,28 @@
   <material>Gazebo/Grey</material>
 </gazebo>
+<!-- <gazebo reference="l_shoulder"> -->
+<!--     <material>Gazebo/White</material> -->
+<!-- </gazebo> -->
+<!-- <gazebo reference="l_shoulder_x"> -->
+<!--     <material>Gazebo/White</material> -->
+<!-- </gazebo> -->
+<!-- <gazebo reference="l_upper_arm"> -->
+<!--     <material>Gazebo/White</material> -->
+<!-- </gazebo> -->
+<!-- <gazebo reference="l_forearm"> -->
+<!--     <material>Gazebo/White</material> -->
+<!-- </gazebo> -->
+<!-- <gazebo reference="l_wrist"> -->
+<!--     <material>Gazebo/White</material> -->
+<!-- </gazebo> -->
+<!-- <gazebo reference="l_wrist2hand"> -->
+<!--     <material>Gazebo/White</material> -->
+<!-- </gazebo> -->
+<!-- <gazebo reference="l_gripper_thumb"> -->
+<!--     <material>Gazebo/White</material> -->
+<!-- </gazebo> -->
+<!-- <gazebo reference="l_gripper_finger"> -->
+<!--     <material>Gazebo/White</material> -->
+<!-- </gazebo> -->
 <link name="torso">
     <inertial>
@@ -37,5 +74,5 @@
         <origin xyz="0.0 0.0 0.0" rpy="0.0 0.0 0.0"/>
         <geometry>
-            <mesh filename="package://reachy_description_ros2/meshes/torso.dae"/>
+            <mesh filename="file://$(find reachy_description_ros2)/meshes/torso.dae"/>
         </geometry>
     </visual>
@@ -58,5 +95,6 @@
         <origin xyz="0.0 0.0 0.0" rpy="0.0 0.0 0.0"/>
         <geometry>
-            <mesh filename="package://reachy_description_ros2/meshes/head.dae"/>
+            <!-- <mesh filename="file://$(find reachy_description_ros2)/meshes/head.dae"/> -->
+            <mesh filename="file://$(find reachy_description_ros2)/meshes/head.dae"/>
         </geometry>
     </visual>
@@ -68,4 +106,7 @@
     </collision>
 </link>
+<!-- <gazebo reference="head"> -->
+<!--   <material>Gazebo/Grey</material> -->
+<!-- </gazebo> -->
 <link name="head_tip"/>
 <link name="l_antenna">
@@ -78,5 +119,5 @@
         <origin xyz="0.0 0.0 0.0" rpy="0.0 0.0 0.0"/>
         <geometry>
-            <mesh filename="package://reachy_description_ros2/meshes/antenna.dae"/>
+            <mesh filename="file://$(find reachy_description_ros2)/meshes/antenna.dae"/>
         </geometry>
     </visual>
@@ -97,5 +138,5 @@
         <origin xyz="0.0 0.0 0.0" rpy="0.0 0.0 0.0"/>
         <geometry>
-            <mesh filename="package://reachy_description_ros2/meshes/antenna.dae"/>
+            <mesh filename="file://$(find reachy_description_ros2)/meshes/antenna.dae"/>
         </geometry>
     </visual>
@@ -119,5 +160,5 @@
         <origin xyz="0.0 0.04 0.0" rpy="1.57 1.57 0.0"/>
         <geometry>
-            <mesh filename="package://reachy_description_ros2/meshes/shoulder.dae"/>
+            <mesh filename="file://$(find reachy_description_ros2)/meshes/shoulder.dae"/>
         </geometry>
     </visual>
@@ -138,5 +179,5 @@
         <origin xyz="0.0 0.0 0.0" rpy="0.0 0.0 0.0"/>
         <geometry>
-            <mesh filename="package://reachy_description_ros2/meshes/shoulder_x.dae"/>
+            <mesh filename="file://$(find reachy_description_ros2)/meshes/shoulder_x.dae"/>
         </geometry>
     </visual>
@@ -157,5 +198,5 @@
         <origin xyz="0.0 0.0 -0.0526" rpy="0.0 0.0 0.0"/>
         <geometry>
-            <mesh filename="package://reachy_description_ros2/meshes/upper_arm.dae"/>
+            <mesh filename="file://$(find reachy_description_ros2)/meshes/upper_arm.dae"/>
         </geometry>
     </visual>
@@ -176,5 +217,5 @@
         <origin xyz="0.0 0.0 0.0" rpy="0.0 0.0 0.0"/>
         <geometry>
-            <mesh filename="package://reachy_description_ros2/meshes/forearm.dae"/>
+            <mesh filename="file://$(find reachy_description_ros2)/meshes/forearm.dae"/>
         </geometry>
     </visual>
@@ -195,5 +236,5 @@
         <origin xyz="0.0 0.0 -0.100" rpy="0.0 0.0 0.0"/>
         <geometry>
-            <mesh filename="package://reachy_description_ros2/meshes/wrist.dae"/>
+            <mesh filename="file://$(find reachy_description_ros2)/meshes/wrist.dae"/>
         </geometry>
     </visual>
@@ -214,5 +255,5 @@
         <origin xyz="0.0 0.0 0.0" rpy="0.0 0.0 0.0"/>
         <geometry>
-            <mesh filename="package://reachy_description_ros2/meshes/wrist2hand.dae"/>
+            <mesh filename="file://$(find reachy_description_ros2)/meshes/wrist2hand.dae"/>
         </geometry>
     </visual>
@@ -226,12 +267,14 @@
 <link name="r_gripper_thumb">
     <inertial>
-        <origin xyz="0.032 -0.008 0.0" rpy="0.0 1.57 0.0"/>
+        <!-- <origin xyz="0.032 -0.008 0.0" rpy="0.0 1.57 0.0"/> -->
+        <origin xyz="0.0 -0.008 0.0" rpy="0.0 1.57 0.0"/>
         <mass value="0.173"/>
-        <inertia ixx="1.083e-4" ixy="-3.476e-5" ixz="1.331e-6" iyy="1.421e-4" iyz="6.730e-7" izz="2.112e-4"/>
+        <!-- <inertia ixx="1.083e-4" ixy="-3.476e-5" ixz="1.331e-6" iyy="1.421e-4" iyz="6.730e-7" izz="2.112e-4"/> -->
+        <inertia ixx="0.0001" izz="0.0001" iyy="0.0001" ixy="0" ixz="0" iyz="0" />
     </inertial>
     <visual name="">
         <origin xyz="0.0 0.0 0.0" rpy="0.0 1.57 0.0"/>
         <geometry>
-            <mesh filename="package://reachy_description_ros2/meshes/r_gripper_thumb.dae"/>
+            <mesh filename="file://$(find reachy_description_ros2)/meshes/r_gripper_thumb.dae"/>
         </geometry>
     </visual>
@@ -245,12 +288,14 @@
 <link name="r_gripper_finger">
     <inertial>
-        <origin xyz="-0.005 -0.043 -0.0" rpy="0.0 1.57 0.0"/>
+        <!-- <origin xyz="-0.005 -0.043 -0.0" rpy="0.0 1.57 0.0"/> -->
+        <origin xyz="-0.00 -0.005 -0.0" rpy="1.57 0.0 1.57"/>
         <mass value="0.035"/>
-        <inertia ixx="9.166e-5" ixy="-6.559e-6" ixz="-3.952e-8" iyy="1.062e-5" iyz="5.276e-9" izz="8.704e-5"/>
+        <!-- <inertia ixx="9.166e-5" ixy="-6.559e-6" ixz="-3.952e-8" iyy="1.062e-5" iyz="5.276e-9" izz="8.704e-5"/> -->
+        <inertia ixx="0.00005" izz="0.00005" iyy="0.00005" ixy="0" ixz="0" iyz="0" />
     </inertial>
     <visual name="">
         <origin xyz="0.0 0.0 0.0" rpy="0.0 1.57 0.0"/>
         <geometry>
-            <mesh filename="package://reachy_description_ros2/meshes/r_gripper_finger.dae"/>
+            <mesh filename="file://$(find reachy_description_ros2)/meshes/r_gripper_finger.dae"/>
         </geometry>
     </visual>
@@ -268,5 +313,5 @@
 <link name="l_shoulder">
     <inertial>
-        <origin xyz="-0.016 0.044 0.0" rpy="-1.57 1.57 0.0"/>
+        <origin xyz="-0.016 -0.036 0.0" rpy="-1.57 1.57 0.0"/>
         <mass value="0.053"/>
         <inertia ixx="3.308e-4" ixy="9.972e-8" ixz="-2.037e-9" iyy="4.650e-5" iyz="2.113e-6" izz="3.545e-5"/>
@@ -275,5 +320,5 @@
         <origin xyz="0.0 -0.04 0.0" rpy="-1.57 1.57 0.0"/>
         <geometry>
-            <mesh filename="package://reachy_description_ros2/meshes/shoulder.dae"/>
+            <mesh filename="file://$(find reachy_description_ros2)/meshes/shoulder.dae"/>
         </geometry>
     </visual>
@@ -294,5 +339,5 @@
         <origin xyz="0.0 0.0 0.0" rpy="0.0 0.0 0.0"/>
         <geometry>
-            <mesh filename="package://reachy_description_ros2/meshes/shoulder_x.dae"/>
+            <mesh filename="file://$(find reachy_description_ros2)/meshes/shoulder_x.dae"/>
         </geometry>
     </visual>
@@ -313,5 +358,5 @@
         <origin xyz="0.0 0.0 -0.0526" rpy="0.0 0.0 0.0"/>
         <geometry>
-            <mesh filename="package://reachy_description_ros2/meshes/upper_arm.dae"/>
+            <mesh filename="file://$(find reachy_description_ros2)/meshes/upper_arm.dae"/>
         </geometry>
     </visual>
@@ -332,5 +377,5 @@
         <origin xyz="0.0 0.0 0.0" rpy="0.0 0.0 0.0"/>
         <geometry>
-            <mesh filename="package://reachy_description_ros2/meshes/forearm.dae"/>
+            <mesh filename="file://$(find reachy_description_ros2)/meshes/forearm.dae"/>
         </geometry>
     </visual>
@@ -351,5 +396,5 @@
         <origin xyz="0.0 0.0 -0.1" rpy="0.0 0.0 0.0"/>
         <geometry>
-            <mesh filename="package://reachy_description_ros2/meshes/wrist.dae"/>
+            <mesh filename="file://$(find reachy_description_ros2)/meshes/wrist.dae"/>
         </geometry>
     </visual>
@@ -370,5 +415,5 @@
         <origin xyz="0.0 0.0 0.0" rpy="0.0 0.0 0.0"/>
         <geometry>
-            <mesh filename="package://reachy_description_ros2/meshes/wrist2hand.dae"/>
+            <mesh filename="file://$(find reachy_description_ros2)/meshes/wrist2hand.dae"/>
         </geometry>
     </visual>
@@ -382,12 +427,14 @@
 <link name="l_gripper_thumb">
     <inertial>
-        <origin xyz="0.032 0.008 0.0" rpy="0.0 1.57 0.0"/>
+        <!-- <origin xyz="0.032 0.008 0.0" rpy="0.0 1.57 0.0"/> -->
+        <origin xyz="0.0 0.008 0.0" rpy="0.0 1.57 0.0"/>
         <mass value="0.173"/>
-        <inertia ixx="1.088e+5" ixy="3.479e+4" ixz="1.357e+3" iyy="1.422e+5" iyz="-7.930e+2" izz="2.116e+5"/>
+        <!-- <inertia ixx="1.088e+5" ixy="3.479e+4" ixz="1.357e+3" iyy="1.422e+5" iyz="-7.930e+2" izz="2.116e+5"/> -->
+        <inertia ixx="0.0001" izz="0.0001" iyy="0.0001" ixy="0" ixz="0" iyz="0" />
     </inertial>
     <visual name="">
         <origin xyz="0.0 0.0 0.0" rpy="0.0 1.57 0.0"/>
         <geometry>
-            <mesh filename="package://reachy_description_ros2/meshes/l_gripper_thumb.dae"/>
+            <mesh filename="file://$(find reachy_description_ros2)/meshes/l_gripper_thumb.dae"/>
         </geometry>
     </visual>
@@ -401,12 +448,14 @@
 <link name="l_gripper_finger">
     <inertial>
-        <origin xyz="0.005 -0.043 0.0" rpy="0.0 1.57 0.0"/>
+        <!-- <origin xyz="0.005 -0.043 0.0" rpy="0.0 1.57 0.0"/> -->
+        <origin xyz="-0.00 0.005 -0.0" rpy="1.57 0.0 1.57"/>
         <mass value="0.035"/>
-        <inertia ixx="9.165e-5" ixy="6.559e-6" ixz="3.609e-10" iyy="1.062e-5" iyz="4.666e-9" izz="8.705e-5"/>
+        <!-- <inertia ixx="9.165e-5" ixy="6.559e-6" ixz="3.609e-10" iyy="1.062e-5" iyz="4.666e-9" izz="8.705e-5"/> -->
+        <inertia ixx="0.00005" izz="0.00005" iyy="0.00005" ixy="0" ixz="0" iyz="0" />
     </inertial>
     <visual name="">
         <origin xyz="0.0 0.0 0.0" rpy="0.0 1.57 0.0"/>
         <geometry>
-            <mesh filename="package://reachy_description_ros2/meshes/l_gripper_finger.dae"/>
+            <mesh filename="file://$(find reachy_description_ros2)/meshes/l_gripper_finger.dae"/>
         </geometry>
     </visual>
@@ -432,5 +481,5 @@
 </joint>
 <xacro:if value="$(arg head)">
-<joint name="r_antenna" type="revolute">
+<joint name="r_antenna_joint" type="revolute">
     <origin xyz="-0.052 -0.057 0.086" rpy="-0.166 -1.054 1.11"/>
     <parent link="head"/>
@@ -438,6 +487,7 @@
     <axis xyz="0 0 1"/>
    <limit lower="-2.618" upper="2.618" effort="10." velocity="0.0"/>
-</joint>
-<joint name="l_antenna" type="revolute">
+    <dynamics damping="${damping}" friction="${friction}" />
+</joint>
+<joint name="l_antenna_joint" type="revolute">
     <origin xyz="-0.052 0.057 0.086" rpy="0.166 -1.054 -1.11"/>
     <parent link="head"/>
@@ -445,4 +495,5 @@
     <axis xyz="0 0 1"/>
    <limit lower="-2.618" upper="2.618" effort="10." velocity="0.0"/>
+    <dynamics damping="${damping}" friction="${friction}" />
 </joint>
 </xacro:if>
@@ -455,4 +506,5 @@
     <axis xyz="0 1 0"/>
    <limit lower="-2.618" upper="1.57" effort="10." velocity="0.0"/>
+    <dynamics damping="${damping}" friction="${friction}" />
 </joint>
 <joint name="r_shoulder_roll" type="revolute">
@@ -462,4 +514,5 @@
     <axis xyz="1 0 0"/>
    <limit lower="-3.14" upper="0.174" effort="10." velocity="0.0"/>
+    <dynamics damping="${damping}" friction="${friction}" />
 </joint>
 <joint name="r_arm_yaw" type="revolute">
@@ -469,4 +522,5 @@
     <axis xyz="0 0 1"/>
    <limit lower="-1.57" upper="1.57" effort="10." velocity="0.0"/>
+    <dynamics damping="${damping}" friction="${friction}" />
 </joint>
 <joint name="r_elbow_pitch" type="revolute">
@@ -476,4 +530,5 @@
     <axis xyz="0 1 0"/>
    <limit lower="-2.182" upper="0" effort="10." velocity="0.0"/>
+    <dynamics damping="${damping}" friction="${friction}" />
 </joint>
 <joint name="r_forearm_yaw" type="revolute">
@@ -483,4 +538,5 @@
     <axis xyz="0 0 1"/>
    <limit lower="-1.745" upper="1.745" effort="10." velocity="0.0"/>
+    <dynamics damping="${damping}" friction="${friction}" />
 </joint>
 <joint name="r_wrist_pitch" type="revolute">
@@ -490,4 +546,5 @@
     <axis xyz="0 1 0"/>
    <limit lower="-0.785" upper="0.785" effort="10." velocity="0.0"/>
+    <dynamics damping="${damping}" friction="${friction}" />
 </joint>
 <joint name="r_wrist_roll" type="revolute">
@@ -497,4 +554,5 @@
     <axis xyz="1 0 0"/>
    <limit lower="-0.785" upper="0.785" effort="10." velocity="0.0"/>
+    <dynamics damping="${damping}" friction="${friction}" />
 </joint>
 <joint name="r_gripper" type="revolute">
@@ -504,4 +562,5 @@
     <axis xyz="1 0 0"/>
    <limit lower="-1.2" upper="0.35" effort="10." velocity="0.0"/>
+    <dynamics damping="${damping}" friction="${friction}" />
 </joint>
 <joint name="r_tip" type="fixed">
@@ -519,4 +578,5 @@
     <axis xyz="0 1 0"/>
    <limit lower="-2.618" upper="1.57" effort="10." velocity="0.0"/>
+    <dynamics damping="${damping}" friction="${friction}" />
 </joint>
 <joint name="l_shoulder_roll" type="revolute">
@@ -526,4 +586,5 @@
     <axis xyz="1 0 0"/>
    <limit lower="-0.174" upper="3.14" effort="10." velocity="0.0"/>
+    <dynamics damping="${damping}" friction="${friction}" />
 </joint>
 <joint name="l_arm_yaw" type="revolute">
@@ -533,4 +594,5 @@
     <axis xyz="0 0 1"/>
    <limit lower="-1.57" upper="1.57" effort="10." velocity="0.0"/>
+    <dynamics damping="${damping}" friction="${friction}" />
 </joint>
 <joint name="l_elbow_pitch" type="revolute">
@@ -540,4 +602,5 @@
     <axis xyz="0 1 0"/>
    <limit lower="-2.182" upper="0" effort="10." velocity="0.0"/>
+    <dynamics damping="${damping}" friction="${friction}" />
 </joint>
 <joint name="l_forearm_yaw" type="revolute">
@@ -547,4 +610,5 @@
     <axis xyz="0 0 1"/>
    <limit lower="-1.745" upper="1.745" effort="10." velocity="0.0"/>
+    <dynamics damping="${damping}" friction="${friction}" />
 </joint>
 <joint name="l_wrist_pitch" type="revolute">
@@ -554,4 +618,5 @@
     <axis xyz="0 1 0"/>
    <limit lower="-0.785" upper="0.785" effort="10." velocity="0.0"/>
+    <dynamics damping="${damping}" friction="${friction}" />
 </joint>
 <joint name="l_wrist_roll" type="revolute">
@@ -561,4 +626,5 @@
     <axis xyz="1 0 0"/>
    <limit lower="-0.785" upper="0.785" effort="10." velocity="0.0"/>
+    <dynamics damping="${damping}" friction="${friction}" />
 </joint>
 <joint name="l_gripper" type="revolute">
@@ -568,4 +634,5 @@
     <axis xyz="1 0 0"/>
    <limit lower="-0.35" upper="1.2" effort="10." velocity="0.0"/>
+    <dynamics damping="${damping}" friction="${friction}" />
 </joint>
 <joint name="l_tip" type="fixed">
@@ -592,4 +659,5 @@
     <axis xyz="1 0 0"/>
    <limit lower="-0.8" upper="0.8" effort="10." velocity="0.0"/>
+    <dynamics damping="${damping}" friction="${friction}" />
 </joint>
 <link name="head_x" >
@@ -606,4 +674,5 @@
     <axis xyz="0 1 0"/>
    <limit lower="-0.8" upper="1.13" effort="10." velocity="0.0"/>
+    <dynamics damping="${damping}" friction="${friction}" />
 </joint>
 <link name="head_y" >
@@ -620,4 +689,5 @@
     <axis xyz="0 0 1"/>
    <limit lower="-2.79" upper="2.79" effort="10." velocity="0.0"/>
+    <dynamics damping="${damping}" friction="${friction}" />
 </joint>
 <link name="head_z" >
@@ -648,5 +718,5 @@
         <origin xyz="0.0 0.0 0.0" rpy="0.0 0.0 0.5236"/>
         <geometry>
-            <mesh filename="package://reachy_description_ros2/meshes/orbita_arm.dae"/>
+            <mesh filename="file://$(find reachy_description_ros2)/meshes/orbita_arm.dae"/>
         </geometry>
     </visual>
@@ -667,5 +737,5 @@
         <origin xyz="0.0 0.0 0.0" rpy="0.0 0.0 2.618"/>
         <geometry>
-            <mesh filename="package://reachy_description_ros2/meshes/orbita_arm.dae"/>
+            <mesh filename="file://$(find reachy_description_ros2)/meshes/orbita_arm.dae"/>
         </geometry>
     </visual>
@@ -686,5 +756,5 @@
         <origin xyz="0.0 0.0 0.0" rpy="0.0 0.0 -1.57"/>
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
File: urdf/reachy_ros2_control.xacro (robot description, xacro)
@@ -5,5 +5,6 @@
         <ros2_control name="${name}" type="system">
             <hardware>
-                <plugin>fake_components/GenericSystem</plugin>
+                <!-- <plugin>fake_components/GenericSystem</plugin> -->
+		<plugin>gazebo_ros2_control/GazeboSystem</plugin>
             </hardware>
             <joint name="orbita_roll">
@@ -73,6 +74,6 @@
                 <state_interface name="velocity"/>
             </joint>
-            <joint name="l_antenna">
-                <param name="initial_position">${initial_positions['l_antenna']}</param>
+            <joint name="l_antenna_joint">
+                <param name="initial_position">${initial_positions['l_antenna_joint']}</param>
                 <command_interface name="position" />
                 <state_interface name="position"/>
@@ -127,6 +128,6 @@
                 <state_interface name="velocity"/>
             </joint>
-            <joint name="r_antenna">
-                <param name="initial_position">${initial_positions['r_antenna']}</param>
+            <joint name="r_antenna_joint">
+                <param name="initial_position">${initial_positions['r_antenna_joint']}</param>
                 <command_interface name="position" />
                 <state_interface name="position"/>

Commit message: Rename antenna_joint to antenna.

File: urdf/reachy.URDF (robot description, URDF)
Before this commit: robot reachy, 31 links, 30 joints
Joints:
- removed joint l_antenna_joint
- removed joint r_antenna_joint
- added joint l_antenna: type revolute, parent head, child l_antenna_link, origin xyz=-0.052 0.057 0.086 rpy=0.166 -1.054 -1.11, axis 0 0 1, limit lower=-2.618 upper=2.618 effort=10. velocity=0.0
- added joint r_antenna: type revolute, parent head, child r_antenna_link, origin xyz=-0.052 -0.057 0.086 rpy=-0.166 -1.054 1.11, axis 0 0 1, limit lower=-2.618 upper=2.618 effort=10. velocity=0.0

File: urdf/reachy.URDF.xacro (robot description, xacro)
@@ -481,5 +481,5 @@
 </joint>
 <xacro:if value="$(arg head)">
-<joint name="r_antenna_joint" type="revolute">
+<joint name="r_antenna" type="revolute">
     <origin xyz="-0.052 -0.057 0.086" rpy="-0.166 -1.054 1.11"/>
     <parent link="head"/>
@@ -489,5 +489,5 @@
     <dynamics damping="${damping}" friction="${friction}" />
 </joint>
-<joint name="l_antenna_joint" type="revolute">
+<joint name="l_antenna" type="revolute">
     <origin xyz="-0.052 0.057 0.086" rpy="0.166 -1.054 -1.11"/>
     <parent link="head"/>

File: urdf/reachy_ros2_control.xacro (robot description, xacro)
@@ -74,6 +74,6 @@
                 <state_interface name="velocity"/>
             </joint>
-            <joint name="l_antenna_joint">
-                <param name="initial_position">${initial_positions['l_antenna_joint']}</param>
+            <joint name="l_antenna">
+                <param name="initial_position">${initial_positions['l_antenna']}</param>
                 <command_interface name="position" />
                 <state_interface name="position"/>
@@ -128,6 +128,6 @@
                 <state_interface name="velocity"/>
             </joint>
-            <joint name="r_antenna_joint">
-                <param name="initial_position">${initial_positions['r_antenna_joint']}</param>
+            <joint name="r_antenna">
+                <param name="initial_position">${initial_positions['r_antenna']}</param>
                 <command_interface name="position" />
                 <state_interface name="position"/>
