Commit message: Use neck instead of orbita in joint names.

File: urdf/reachy.URDF (robot description, URDF)
Before this commit: robot reachy, 31 links, 30 joints
Links:
- removed link bottom_orbita_arm
- removed link middle_orbita_arm
- removed link top_orbita_arm
- added link bottom_neck_arm; collision cylinder length=0.0 radius=0.0; visual mesh filename=package://reachy_description_ros2/meshes/orbita_arm.dae
- added link middle_neck_arm; collision cylinder length=0.0 radius=0.0; visual mesh filename=package://reachy_description_ros2/meshes/orbita_arm.dae
- added link top_neck_arm; collision cylinder length=0.0 radius=0.0; visual mesh filename=package://reachy_description_ros2/meshes/orbita_arm.dae
Joints:
- removed joint orbita_bottom
- removed joint orbita_fixed
- removed joint orbita_middle
- removed joint orbita_pitch
- removed joint orbita_roll
- removed joint orbita_top
- removed joint orbita_yaw
- added joint neck_bottom: type fixed, parent torso, child bottom_neck_arm, origin xyz=0.0067 0.0 0.0478 rpy=0 0.174 0
- added joint neck_fixed: type fixed, parent head_z, child head, origin xyz=0 0 0 rpy=0.0 0.0 0.0
- added joint neck_middle: type fixed, parent torso, child middle_neck_arm, origin xyz=0.0067 0.0 0.0478 rpy=0 0.174 0
- added joint neck_pitch: type revolute, parent head_x, child head_y, origin xyz=0 0 0 rpy=0.0 0.0 0.0, axis 0 1 0, limit lower=-0.8 upper=1.13 effort=10. velocity=0.0
- added joint neck_roll: type revolute, parent torso, child head_x, origin xyz=0.015 0.0 0.095 rpy=0 0.174 0, axis 1 0 0, limit lower=-0.8 upper=0.8 effort=10. velocity=0.0
- added joint neck_top: type fixed, parent torso, child top_neck_arm, origin xyz=0.0067 0.0 0.0478 rpy=0 0.174 0
- added joint neck_yaw: type revolute, parent head_y, child head_z, origin xyz=0 0 0 rpy=0.0 0.0 0.0, axis 0 0 1, limit lower=-2.79 upper=2.79 effort=10. velocity=0.0

File: urdf/reachy.URDF.xacro (robot description, xacro)
@@ -653,5 +653,5 @@
 <!-- ...with a ball orbita joint -->
 <xacro:if value="$(arg head)">
-<joint name="orbita_roll" type="revolute">
+<joint name="neck_roll" type="revolute">
     <origin xyz="0.015 0.0 0.095" rpy="0 0.174 0" />
     <parent link="torso"/>
@@ -668,5 +668,5 @@
 </inertial>
 </link>
-<joint name="orbita_pitch" type="revolute">
+<joint name="neck_pitch" type="revolute">
     <origin xyz="0 0 0" rpy="0.0 0.0 0.0"/>
     <parent link="head_x"/>
@@ -683,5 +683,5 @@
 </inertial>
 </link>
-<joint name="orbita_yaw" type="revolute">
+<joint name="neck_yaw" type="revolute">
     <origin xyz="0 0 0" rpy="0.0 0.0 0.0"/>
     <parent link="head_y"/>
@@ -698,5 +698,5 @@
 </inertial>
 </link>
-<joint name="orbita_fixed" type="fixed">
+<joint name="neck_fixed" type="fixed">
     <origin xyz="0 0 0" rpy="0.0 0.0 0.0"/>
     <parent link="head_z" />
@@ -709,10 +709,10 @@
 </joint>
 <!-- Fixed Orbita Arms Visuals -->
-<joint name="orbita_top" type="fixed">
+<joint name="neck_top" type="fixed">
     <origin xyz="0.0067 0.0 0.0478" rpy="0 0.174 0"/>
     <parent link="torso"/>
-    <child link="top_orbita_arm"/>
-</joint>
-<link name="top_orbita_arm">
+    <child link="top_neck_arm"/>
+</joint>
+<link name="top_neck_arm">
     <visual name="">
         <origin xyz="0.0 0.0 0.0" rpy="0.0 0.0 0.5236"/>
@@ -728,10 +728,10 @@
     </collision>
 </link>
-<joint name="orbita_middle" type="fixed">
+<joint name="neck_middle" type="fixed">
     <origin xyz="0.0067 0.0 0.0478" rpy="0 0.174 0"/>
     <parent link="torso"/>
-    <child link="middle_orbita_arm"/>
-</joint>
-<link name="middle_orbita_arm">
+    <child link="middle_neck_arm"/>
+</joint>
+<link name="middle_neck_arm">
     <visual name="">
         <origin xyz="0.0 0.0 0.0" rpy="0.0 0.0 2.618"/>
@@ -747,10 +747,10 @@
     </collision>
 </link>
-<joint name="orbita_bottom" type="fixed">
+<joint name="neck_bottom" type="fixed">
     <origin xyz="0.0067 0.0 0.0478" rpy="0 0.174 0"/>
     <parent link="torso"/>
-    <child link="bottom_orbita_arm"/>
-</joint>
-<link name="bottom_orbita_arm">
+    <child link="bottom_neck_arm"/>
+</joint>
+<link name="bottom_neck_arm">
     <visual name="">
         <origin xyz="0.0 0.0 0.0" rpy="0.0 0.0 -1.57"/>

File: urdf/reachy_ros2_control.xacro (robot description, xacro)
@@ -8,18 +8,18 @@
 		<plugin>gazebo_ros2_control/GazeboSystem</plugin>
             </hardware>
-            <joint name="orbita_roll">
-                <param name="initial_position">${initial_positions['orbita_roll']}</param>
+            <joint name="neck_roll">
+                <param name="initial_position">${initial_positions['neck_roll']}</param>
                 <command_interface name="position" />
                 <state_interface name="position"/>
                 <state_interface name="velocity"/>
             </joint>
-            <joint name="orbita_pitch">
-                <param name="initial_position">${initial_positions['orbita_pitch']}</param>
+            <joint name="neck_pitch">
+                <param name="initial_position">${initial_positions['neck_pitch']}</param>
                 <command_interface name="position" />
                 <state_interface name="position"/>
                 <state_interface name="velocity"/>
             </joint>
-            <joint name="orbita_yaw">
-                <param name="initial_position">${initial_positions['orbita_yaw']}</param>
+            <joint name="neck_yaw">
+                <param name="initial_position">${initial_positions['neck_yaw']}</param>
                 <command_interface name="position" />
                 <state_interface name="position"/>

Commit message: Change deprecated name.

File: urdf/reachy.URDF (robot description, URDF)
Before this commit: robot reachy, 31 links, 30 joints
Links:
- link bottom_neck_arm: geometry collision cylinder length=0.0 radius=0.0; visual mesh filename=package://reachy_description/meshes/orbita_arm.dae
- link head: geometry collision cylinder length=0.15 radius=0.06; visual mesh filename=package://reachy_description/meshes/head.dae
- link l_antenna_link: geometry collision cylinder length=0.0 radius=0.0; visual mesh filename=package://reachy_description/meshes/antenna.dae
- link l_forearm: geometry collision cylinder length=0.09 radius=0.04; visual mesh filename=package://reachy_description/meshes/forearm.dae
- link l_gripper_finger: geometry collision box size=0.1 0.012 0.035; visual mesh filename=package://reachy_description/meshes/l_gripper_finger.dae
- link l_gripper_thumb: geometry collision box size=0.1 0.012 0.035; visual mesh filename=package://reachy_description/meshes/l_gripper_thumb.dae
- link l_shoulder: geometry collision cylinder length=0.09 radius=0.035; visual mesh filename=package://reachy_description/meshes/shoulder.dae
- link l_shoulder_x: geometry collision cylinder length=0.04 radius=0.035; visual mesh filename=package://reachy_description/meshes/shoulder_x.dae
- link l_upper_arm: geometry collision cylinder length=0.25 radius=0.04; visual mesh filename=package://reachy_description/meshes/upper_arm.dae
- link l_wrist: geometry collision cylinder length=0.14 radius=0.035; visual mesh filename=package://reachy_description/meshes/wrist.dae
- link l_wrist2hand: geometry collision cylinder length=0.06 radius=0.03; visual mesh filename=package://reachy_description/meshes/wrist2hand.dae
- link middle_neck_arm: geometry collision cylinder length=0.0 radius=0.0; visual mesh filename=package://reachy_description/meshes/orbita_arm.dae
- link r_antenna_link: geometry collision cylinder length=0.0 radius=0.0; visual mesh filename=package://reachy_description/meshes/antenna.dae
- link r_forearm: geometry collision cylinder length=0.09 radius=0.04; visual mesh filename=package://reachy_description/meshes/forearm.dae
- link r_gripper_finger: geometry collision box size=0.1 0.012 0.035; visual mesh filename=package://reachy_description/meshes/r_gripper_finger.dae
- link r_gripper_thumb: geometry collision box size=0.1 0.012 0.035; visual mesh filename=package://reachy_description/meshes/r_gripper_thumb.dae
- link r_shoulder: geometry collision cylinder length=0.09 radius=0.035; visual mesh filename=package://reachy_description/meshes/shoulder.dae
- link r_shoulder_x: geometry collision cylinder length=0.04 radius=0.035; visual mesh filename=package://reachy_description/meshes/shoulder_x.dae
- link r_upper_arm: geometry collision cylinder length=0.25 radius=0.04; visual mesh filename=package://reachy_description/meshes/upper_arm.dae
- link r_wrist: geometry collision cylinder length=0.14 radius=0.035; visual mesh filename=package://reachy_description/meshes/wrist.dae
- link r_wrist2hand: geometry collision cylinder length=0.06 radius=0.03; visual mesh filename=package://reachy_description/meshes/wrist2hand.dae
- link top_neck_arm: geometry collision cylinder length=0.0 radius=0.0; visual mesh filename=package://reachy_description/meshes/orbita_arm.dae
- link torso: geometry collision box size=0.11 0.2 0.32; visual mesh filename=package://reachy_description/meshes/torso.dae

File: urdf/reachy.URDF.xacro (robot description, xacro)
@@ -74,5 +74,5 @@
         <origin xyz="0.0 0.0 0.0" rpy="0.0 0.0 0.0"/>
         <geometry>
-            <mesh filename="file://$(find reachy_description_ros2)/meshes/torso.dae"/>
+            <mesh filename="file://$(find reachy_description)/meshes/torso.dae"/>
         </geometry>
     </visual>
@@ -95,6 +95,6 @@
         <origin xyz="0.0 0.0 0.0" rpy="0.0 0.0 0.0"/>
         <geometry>
-            <!-- <mesh filename="file://$(find reachy_description_ros2)/meshes/head.dae"/> -->
-            <mesh filename="file://$(find reachy_description_ros2)/meshes/head.dae"/>
+            <!-- <mesh filename="file://$(find reachy_description)/meshes/head.dae"/> -->
+            <mesh filename="file://$(find reachy_description)/meshes/head.dae"/>
         </geometry>
     </visual>
@@ -119,5 +119,5 @@
         <origin xyz="0.0 0.0 0.0" rpy="0.0 0.0 0.0"/>
         <geometry>
-            <mesh filename="file://$(find reachy_description_ros2)/meshes/antenna.dae"/>
+            <mesh filename="file://$(find reachy_description)/meshes/antenna.dae"/>
         </geometry>
     </visual>
@@ -138,5 +138,5 @@
         <origin xyz="0.0 0.0 0.0" rpy="0.0 0.0 0.0"/>
         <geometry>
-            <mesh filename="file://$(find reachy_description_ros2)/meshes/antenna.dae"/>
+            <mesh filename="file://$(find reachy_description)/meshes/antenna.dae"/>
         </geometry>
     </visual>
@@ -160,5 +160,5 @@
         <origin xyz="0.0 0.04 0.0" rpy="1.57 1.57 0.0"/>
         <geometry>
-            <mesh filename="file://$(find reachy_description_ros2)/meshes/shoulder.dae"/>
+            <mesh filename="file://$(find reachy_description)/meshes/shoulder.dae"/>
         </geometry>
     </visual>
@@ -179,5 +179,5 @@
         <origin xyz="0.0 0.0 0.0" rpy="0.0 0.0 0.0"/>
         <geometry>
-            <mesh filename="file://$(find reachy_description_ros2)/meshes/shoulder_x.dae"/>
+            <mesh filename="file://$(find reachy_description)/meshes/shoulder_x.dae"/>
         </geometry>
     </visual>
@@ -198,5 +198,5 @@
         <origin xyz="0.0 0.0 -0.0526" rpy="0.0 0.0 0.0"/>
         <geometry>
-            <mesh filename="file://$(find reachy_description_ros2)/meshes/upper_arm.dae"/>
+            <mesh filename="file://$(find reachy_description)/meshes/upper_arm.dae"/>
         </geometry>
     </visual>
@@ -217,5 +217,5 @@
         <origin xyz="0.0 0.0 0.0" rpy="0.0 0.0 0.0"/>
         <geometry>
-            <mesh filename="file://$(find reachy_description_ros2)/meshes/forearm.dae"/>
+            <mesh filename="file://$(find reachy_description)/meshes/forearm.dae"/>
         </geometry>
     </visual>
@@ -236,5 +236,5 @@
         <origin xyz="0.0 0.0 -0.100" rpy="0.0 0.0 0.0"/>
         <geometry>
-            <mesh filename="file://$(find reachy_description_ros2)/meshes/wrist.dae"/>
+            <mesh filename="file://$(find reachy_description)/meshes/wrist.dae"/>
         </geometry>
     </visual>
@@ -255,5 +255,5 @@
         <origin xyz="0.0 0.0 0.0" rpy="0.0 0.0 0.0"/>
         <geometry>
-            <mesh filename="file://$(find reachy_description_ros2)/meshes/wrist2hand.dae"/>
+            <mesh filename="file://$(find reachy_description)/meshes/wrist2hand.dae"/>
         </geometry>
     </visual>
@@ -276,5 +276,5 @@
         <origin xyz="0.0 0.0 0.0" rpy="0.0 1.57 0.0"/>
         <geometry>
-            <mesh filename="file://$(find reachy_description_ros2)/meshes/r_gripper_thumb.dae"/>
+            <mesh filename="file://$(find reachy_description)/meshes/r_gripper_thumb.dae"/>
         </geometry>
     </visual>
@@ -297,5 +297,5 @@
         <origin xyz="0.0 0.0 0.0" rpy="0.0 1.57 0.0"/>
         <geometry>
-            <mesh filename="file://$(find reachy_description_ros2)/meshes/r_gripper_finger.dae"/>
+            <mesh filename="file://$(find reachy_description)/meshes/r_gripper_finger.dae"/>
         </geometry>
     </visual>
@@ -320,5 +320,5 @@
         <origin xyz="0.0 -0.04 0.0" rpy="-1.57 1.57 0.0"/>
         <geometry>
-            <mesh filename="file://$(find reachy_description_ros2)/meshes/shoulder.dae"/>
+            <mesh filename="file://$(find reachy_description)/meshes/shoulder.dae"/>
         </geometry>
     </visual>
@@ -339,5 +339,5 @@
         <origin xyz="0.0 0.0 0.0" rpy="0.0 0.0 0.0"/>
         <geometry>
-            <mesh filename="file://$(find reachy_description_ros2)/meshes/shoulder_x.dae"/>
+            <mesh filename="file://$(find reachy_description)/meshes/shoulder_x.dae"/>
         </geometry>
     </visual>
@@ -358,5 +358,5 @@
         <origin xyz="0.0 0.0 -0.0526" rpy="0.0 0.0 0.0"/>
         <geometry>
-            <mesh filename="file://$(find reachy_description_ros2)/meshes/upper_arm.dae"/>
+            <mesh filename="file://$(find reachy_description)/meshes/upper_arm.dae"/>
         </geometry>
     </visual>
@@ -377,5 +377,5 @@
         <origin xyz="0.0 0.0 0.0" rpy="0.0 0.0 0.0"/>
         <geometry>
-            <mesh filename="file://$(find reachy_description_ros2)/meshes/forearm.dae"/>
+            <mesh filename="file://$(find reachy_description)/meshes/forearm.dae"/>
         </geometry>
     </visual>
@@ -396,5 +396,5 @@
         <origin xyz="0.0 0.0 -0.1" rpy="0.0 0.0 0.0"/>
         <geometry>
-            <mesh filename="file://$(find reachy_description_ros2)/meshes/wrist.dae"/>
+            <mesh filename="file://$(find reachy_description)/meshes/wrist.dae"/>
         </geometry>
     </visual>
@@ -415,5 +415,5 @@
         <origin xyz="0.0 0.0 0.0" rpy="0.0 0.0 0.0"/>
         <geometry>
-            <mesh filename="file://$(find reachy_description_ros2)/meshes/wrist2hand.dae"/>
+            <mesh filename="file://$(find reachy_description)/meshes/wrist2hand.dae"/>
         </geometry>
     </visual>
@@ -436,5 +436,5 @@
         <origin xyz="0.0 0.0 0.0" rpy="0.0 1.57 0.0"/>
         <geometry>
-            <mesh filename="file://$(find reachy_description_ros2)/meshes/l_gripper_thumb.dae"/>
+            <mesh filename="file://$(find reachy_description)/meshes/l_gripper_thumb.dae"/>
         </geometry>
     </visual>
@@ -457,5 +457,5 @@
         <origin xyz="0.0 0.0 0.0" rpy="0.0 1.57 0.0"/>
         <geometry>
-            <mesh filename="file://$(find reachy_description_ros2)/meshes/l_gripper_finger.dae"/>
+            <mesh filename="file://$(find reachy_description)/meshes/l_gripper_finger.dae"/>
         </geometry>
     </visual>
@@ -718,5 +718,5 @@
         <origin xyz="0.0 0.0 0.0" rpy="0.0 0.0 0.5236"/>
         <geometry>
-            <mesh filename="file://$(find reachy_description_ros2)/meshes/orbita_arm.dae"/>
+            <mesh filename="file://$(find reachy_description)/meshes/orbita_arm.dae"/>
         </geometry>
     </visual>
@@ -737,5 +737,5 @@
         <origin xyz="0.0 0.0 0.0" rpy="0.0 0.0 2.618"/>
         <geometry>
-            <mesh filename="file://$(find reachy_description_ros2)/meshes/orbita_arm.dae"/>
+            <mesh filename="file://$(find reachy_description)/meshes/orbita_arm.dae"/>
         </geometry>
     </visual>
@@ -756,5 +756,5 @@
         <origin xyz="0.0 0.0 0.0" rpy="0.0 0.0 -1.57"/>
         <geometry>
-            <mesh filename="file://$(find reachy_description_ros2)/meshes/orbita_arm.dae"/>
+            <mesh filename="file://$(find reachy_description)/meshes/orbita_arm.dae"/>
         </geometry>
     </visual>
@@ -787,10 +787,10 @@
       <!-- <robotNamespace>/reachy</robotNamespace> -->
       <!-- <robotSimType>gazebo_ros_control/DefaultRobotHWSim</robotSimType> -->
-      <parameters>$(find reachy_gazebo_ros2)/config/reachy_gazebo_controllers.yaml</parameters>
+      <parameters>$(find reachy_gazebo)/config/reachy_gazebo_controllers.yaml</parameters>
     </plugin>
 </gazebo>
 <!-- Declare transmission/motors -->
-<xacro:arg name="initial_positions_file" default="$(find reachy_description_ros2)/urdf/initial_positions.yaml" />
-<xacro:include filename="$(find reachy_description_ros2)/urdf/reachy_ros2_control.xacro" />
+<xacro:arg name="initial_positions_file" default="$(find reachy_description)/urdf/initial_positions.yaml" />
+<xacro:include filename="$(find reachy_description)/urdf/reachy_ros2_control.xacro" />
 <xacro:reachy_ros2_control name="ReachyFakeSystem" initial_positions_file="$(arg initial_positions_file)"/>
 </robot>
