Commit message: Reproduce changes from broken branch.

File: urdf/reachy.URDF (robot description, URDF)
Before this commit: robot reachy, 31 links, 30 joints
Links:
- removed link bottom_orbita_arm
- removed link l_antenna
- removed link middle_orbita_arm
- removed link r_antenna
- removed link top_orbita_arm
- added link bottom_neck_arm; collision cylinder length=0.0 radius=0.0; visual mesh filename=package://reachy_description/meshes/orbita_arm.dae
- added link l_antenna_link, mass 0.004; collision cylinder length=0.0 radius=0.0; visual mesh filename=package://reachy_description/meshes/antenna.dae
- added link middle_neck_arm; collision cylinder length=0.0 radius=0.0; visual mesh filename=package://reachy_description/meshes/orbita_arm.dae
- added link r_antenna_link, mass 0.004; collision cylinder length=0.0 radius=0.0; visual mesh filename=package://reachy_description/meshes/antenna.dae
- added link top_neck_arm; collision cylinder length=0.0 radius=0.0; visual mesh filename=package://reachy_description/meshes/orbita_arm.dae
Joints:
- removed joint orbita_bottom
- removed joint orbita_fixed
- removed joint orbita_middle
- removed joint orbita_pitch
- removed joint orbita_roll
- removed joint orbita_top
- removed joint orbita_yaw
- added joint neck_bottom: type fixed, parent torso, child bottom_neck_arm, origin xyz=0.0067 0.0 0.0478 rpy=0 0.174 0
- added joint neck_fixed: type fixed, parent head_z, child head, origin xyz=0 0 0 rpy=0.0 0.0 0.0
- added joint neck_middle: type fixed, parent torso, child middle_neck_arm, origin xyz=0.0067 0.0 0.0478 rpy=0 0.174 0
- added joint neck_pitch: type revolute, parent head_x, child head_y, origin xyz=0 0 0 rpy=0.0 0.0 0.0, axis 0 1 0, limit lower=-0.8 upper=1.13 effort=10. velocity=0.0
- added joint neck_roll: type revolute, parent torso, child head_x, origin xyz=0.015 0.0 0.095 rpy=0 0.174 0, axis 1 0 0, limit lower=-0.8 upper=0.8 effort=10. velocity=0.0
- added joint neck_top: type fixed, parent torso, child top_neck_arm, origin xyz=0.0067 0.0 0.0478 rpy=0 0.174 0
- added joint neck_yaw: type revolute, parent head_y, child head_z, origin xyz=0 0 0 rpy=0.0 0.0 0.0, axis 0 0 1, limit lower=-2.79 upper=2.79 effort=10. velocity=0.0
- joint l_antenna: child l_antenna -> l_antenna_link
- joint r_antenna: child r_antenna -> r_antenna_link

File: urdf/reachy.URDF.xacro (robot description, xacro)
@@ -4,6 +4,68 @@
 <xacro:arg name="left_arm" default="true"/>
 <xacro:arg name="right_arm" default="true"/>
+<xacro:arg name="depth_camera" default="true"/>
+<!-- pretty important for stability -->
+<xacro:property name="damping" value="0" />
+<xacro:property name="friction" value="0.1" />
+<xacro:macro name="xmass" params="value"><mass value="${value}" /></xacro:macro>
+<xacro:property name="camera_link" value="0.05" /> <!-- Size of square 'camera' box -->
+<xacro:property name="camera_convergence" value="0.0" /> <!-- convergence angle (rad) of the cameras. 0=parallel-->
+<xacro:macro name="inertial_cuboid" params="mass xyz rpy x_length y_length z_length">
+  <inertial>
+    <xacro:xmass value="${mass}" />
+    <origin rpy="${rpy}" xyz="${xyz}"/>
+    <inertia ixx="${mass * (y_length*y_length + z_length*z_length) / 12}" ixy="0.0" ixz="0.0"
+             iyy="${mass * (x_length*x_length + z_length*z_length) / 12}" iyz="0.0"
+             izz="${mass * (x_length*x_length + y_length*y_length) / 12}" />
+  </inertial>
+</xacro:macro>
 <!-- Torso Link -->
-<link name="pedestal"/>
+  <material name="Grey">
+    <color rgba="0.2 0.2 0.2 1"/>
+  </material>
+<link name="pedestal">
+    <collision>
+        <origin xyz="0 0 0.5" rpy="0 0.0 0" />
+        <geometry>
+            <!-- <box size="0.05 0.05 1" /> -->
+	    <cylinder length="1" radius="0.025"/>
+        </geometry>
+    </collision>
+    <visual name="">
+        <origin xyz="0 0 0.5" rpy="0 0.0 0" />
+        <geometry>
+            <!-- <box size="0.05 0.05 1" /> -->
+	    <cylinder length="1" radius="0.025"/>
+        </geometry>
+	 <material name="Grey"/>
+    </visual>
+</link>
+<gazebo reference="pedestal">
+  <material>Gazebo/Grey</material>
+</gazebo>
+<!-- <gazebo reference="l_shoulder"> -->
+<!--     <material>Gazebo/White</material> -->
+<!-- </gazebo> -->
+<!-- <gazebo reference="l_shoulder_x"> -->
+<!--     <material>Gazebo/White</material> -->
+<!-- </gazebo> -->
+<!-- <gazebo reference="l_upper_arm"> -->
+<!--     <material>Gazebo/White</material> -->
+<!-- </gazebo> -->
+<!-- <gazebo reference="l_forearm"> -->
+<!--     <material>Gazebo/White</material> -->
+<!-- </gazebo> -->
+<!-- <gazebo reference="l_wrist"> -->
+<!--     <material>Gazebo/White</material> -->
+<!-- </gazebo> -->
+<!-- <gazebo reference="l_wrist2hand"> -->
+<!--     <material>Gazebo/White</material> -->
+<!-- </gazebo> -->
+<!-- <gazebo reference="l_gripper_thumb"> -->
+<!--     <material>Gazebo/White</material> -->
+<!-- </gazebo> -->
+<!-- <gazebo reference="l_gripper_finger"> -->
+<!--     <material>Gazebo/White</material> -->
+<!-- </gazebo> -->
 <link name="torso">
     <inertial>
@@ -15,5 +77,5 @@
         <origin xyz="0.0 0.0 0.0" rpy="0.0 0.0 0.0"/>
         <geometry>
-            <mesh filename="package://reachy_description/meshes/torso.dae"/>
+            <mesh filename="file://$(find reachy_description)/meshes/torso.dae"/>
         </geometry>
     </visual>
@@ -36,9 +98,10 @@
         <origin xyz="0.0 0.0 0.0" rpy="0.0 0.0 0.0"/>
         <geometry>
-            <mesh filename="package://reachy_description/meshes/head.dae"/>
-        </geometry>
-    </visual>
-    <collision>
-        <origin xyz="-0.009 -0.002 0.059" rpy="1.57 0.0 0.0"/>
+            <!-- <mesh filename="file://$(find reachy_description)/meshes/head.dae"/> -->
+            <mesh filename="file://$(find reachy_description)/meshes/head.dae"/>
+        </geometry>
+    </visual>
+    <collision>
+        <origin xyz="-0.009 -0.002 0.059" rpy="${pi/2.0} 0.0 0.0"/>
         <geometry>
             <cylinder length="0.15" radius="0.06" />
@@ -46,5 +109,9 @@
     </collision>
 </link>
-<link name="l_antenna">
+<!-- <gazebo reference="head"> -->
+<!--   <material>Gazebo/Grey</material> -->
+<!-- </gazebo> -->
+<link name="head_tip"/>
+<link name="l_antenna_link">
     <inertial>
         <origin xyz="-0.001 0.0 0.008" rpy="0.0 0.0 0.0"/>
@@ -55,5 +122,5 @@
         <origin xyz="0.0 0.0 0.0" rpy="0.0 0.0 0.0"/>
         <geometry>
-            <mesh filename="package://reachy_description/meshes/antenna.dae"/>
+            <mesh filename="file://$(find reachy_description)/meshes/antenna.dae"/>
         </geometry>
     </visual>
@@ -65,5 +132,5 @@
     </collision>
 </link>
-<link name="r_antenna">
+<link name="r_antenna_link">
     <inertial>
         <origin xyz="-0.001 0.0 0.008" rpy="0.0 0.0 0.0"/>
@@ -74,5 +141,5 @@
         <origin xyz="0.0 0.0 0.0" rpy="0.0 0.0 0.0"/>
         <geometry>
-            <mesh filename="package://reachy_description/meshes/antenna.dae"/>
+            <mesh filename="file://$(find reachy_description)/meshes/antenna.dae"/>
         </geometry>
     </visual>
@@ -89,16 +156,16 @@
 <link name="r_shoulder">
     <inertial>
-        <origin xyz="-0.016 0.036 0.0" rpy="1.57 1.57 0.0"/>
+        <origin xyz="-0.016 0.036 0.0" rpy="${pi/2.0} ${pi/2.0} 0.0"/>
         <mass value="0.053"/>
         <inertia ixx="3.308e-4" ixy="9.972e-8" ixz="-2.037e-9" iyy="4.650e-5" iyz="2.113e-6" izz="3.545e-5"/>
     </inertial>
     <visual name="">
-        <origin xyz="0.0 0.04 0.0" rpy="1.57 1.57 0.0"/>
-        <geometry>
-            <mesh filename="package://reachy_description/meshes/shoulder.dae"/>
-        </geometry>
-    </visual>
-    <collision>
-        <origin xyz="0.0 0.04 0.0" rpy="1.57 1.57 0.0"/>
+        <origin xyz="0.0 0.04 0.0" rpy="${pi/2.0} ${pi/2.0} 0.0"/>
+        <geometry>
+            <mesh filename="file://$(find reachy_description)/meshes/shoulder.dae"/>
+        </geometry>
+    </visual>
+    <collision>
+        <origin xyz="0.0 0.04 0.0" rpy="${pi/2.0} ${pi/2.0} 0.0"/>
         <geometry>
             <cylinder length="0.09" radius="0.035" />
@@ -110,10 +177,10 @@
         <origin xyz="-0.0 0.0 -0.019" rpy="0.0 0.0 0.0"/>
         <mass value="0.158"/>
-        <inertia ixx="6.887e+4" ixy="5.393e+0" ixz="-9.155e+2" iyy="7.895e+4" iyz="4.512e-1" izz="4.235e+4"/>
-    </inertial>
-    <visual name="">
-        <origin xyz="0.0 0.0 0.0" rpy="0.0 0.0 0.0"/>
-        <geometry>
-            <mesh filename="package://reachy_description/meshes/shoulder_x.dae"/>
+        <inertia ixx="6.887e-5" ixy="5.393e-9" ixz="-9.155e-7" iyy="7.895e-5" iyz="4.512e-10" izz="4.235e-5"/>
+    </inertial>
+    <visual name="">
+        <origin xyz="0.0 0.0 0.0" rpy="0.0 0.0 0.0"/>
+        <geometry>
+            <mesh filename="file://$(find reachy_description)/meshes/shoulder_x.dae"/>
         </geometry>
     </visual>
@@ -134,5 +201,5 @@
         <origin xyz="0.0 0.0 -0.0526" rpy="0.0 0.0 0.0"/>
         <geometry>
-            <mesh filename="package://reachy_description/meshes/upper_arm.dae"/>
+            <mesh filename="file://$(find reachy_description)/meshes/upper_arm.dae"/>
         </geometry>
     </visual>
@@ -153,5 +220,5 @@
         <origin xyz="0.0 0.0 0.0" rpy="0.0 0.0 0.0"/>
         <geometry>
-            <mesh filename="package://reachy_description/meshes/forearm.dae"/>
+            <mesh filename="file://$(find reachy_description)/meshes/forearm.dae"/>
         </geometry>
     </visual>
@@ -172,5 +239,5 @@
         <origin xyz="0.0 0.0 -0.100" rpy="0.0 0.0 0.0"/>
         <geometry>
-            <mesh filename="package://reachy_description/meshes/wrist.dae"/>
+            <mesh filename="file://$(find reachy_description)/meshes/wrist.dae"/>
         </geometry>
     </visual>
@@ -191,5 +258,5 @@
         <origin xyz="0.0 0.0 0.0" rpy="0.0 0.0 0.0"/>
         <geometry>
-            <mesh filename="package://reachy_description/meshes/wrist2hand.dae"/>
+            <mesh filename="file://$(find reachy_description)/meshes/wrist2hand.dae"/>
         </geometry>
     </visual>
@@ -203,16 +270,18 @@
 <link name="r_gripper_thumb">
     <inertial>
-        <origin xyz="0.032 -0.008 0.0" rpy="0.0 1.57 0.0"/>
+        <!-- <origin xyz="0.032 -0.008 0.0" rpy="0.0 1.57 0.0"/> -->
+        <origin xyz="0.0 -0.008 0.0" rpy="0.0 ${pi/2.0} 0.0"/>
         <mass value="0.173"/>
-        <inertia ixx="1.083e-4" ixy="-3.476e-5" ixz="1.331e-6" iyy="1.421e-4" iyz="6.730e-7" izz="2.112e-4"/>
-    </inertial>
-    <visual name="">
-        <origin xyz="0.0 0.0 0.0" rpy="0.0 1.57 0.0"/>
-        <geometry>
-            <mesh filename="package://reachy_description/meshes/r_gripper_thumb.dae"/>
-        </geometry>
-    </visual>
-    <collision>
-        <origin xyz="0.0 0.02 -0.06" rpy="0.0 1.57 0.0"/>
+        <!-- <inertia ixx="1.083e-4" ixy="-3.476e-5" ixz="1.331e-6" iyy="1.421e-4" iyz="6.730e-7" izz="2.112e-4"/> -->
+        <inertia ixx="0.0001" izz="0.0001" iyy="0.0001" ixy="0" ixz="0" iyz="0" />
+    </inertial>
+    <visual name="">
+        <origin xyz="0.0 0.0 0.0" rpy="0.0 ${pi/2.0} 0.0"/>
+        <geometry>
+            <mesh filename="file://$(find reachy_description)/meshes/r_gripper_thumb.dae"/>
+        </geometry>
+    </visual>
+    <collision>
+        <origin xyz="0.0 0.02 -0.06" rpy="0.0 ${pi/2.0} 0.0"/>
         <geometry>
             <box size="0.1 0.012 0.035" />
@@ -222,16 +291,18 @@
 <link name="r_gripper_finger">
     <inertial>
-        <origin xyz="-0.005 -0.043 -0.0" rpy="0.0 1.57 0.0"/>
+        <!-- <origin xyz="-0.005 -0.043 -0.0" rpy="0.0 1.57 0.0"/> -->
+        <origin xyz="-0.00 -0.005 -0.0" rpy="${pi/2.0} 0.0 ${pi/2.0}"/>
         <mass value="0.035"/>
-        <inertia ixx="9.166e-5" ixy="-6.559e-6" ixz="-3.952e-8" iyy="1.062e-5" iyz="5.276e-9" izz="8.704e-5"/>
-    </inertial>
-    <visual name="">
-        <origin xyz="0.0 0.0 0.0" rpy="0.0 1.57 0.0"/>
-        <geometry>
-            <mesh filename="package://reachy_description/meshes/r_gripper_finger.dae"/>
-        </geometry>
-    </visual>
-    <collision>
-        <origin xyz="0.0 -0.01 -0.02" rpy="0.0 1.57 0.0"/>
+        <!-- <inertia ixx="9.166e-5" ixy="-6.559e-6" ixz="-3.952e-8" iyy="1.062e-5" iyz="5.276e-9" izz="8.704e-5"/> -->
+        <inertia ixx="0.00005" izz="0.00005" iyy="0.00005" ixy="0" ixz="0" iyz="0" />
+    </inertial>
+    <visual name="">
+        <origin xyz="0.0 0.0 0.0" rpy="0.0 ${pi/2.0} 0.0"/>
+        <geometry>
+            <mesh filename="file://$(find reachy_description)/meshes/r_gripper_finger.dae"/>
+        </geometry>
+    </visual>
+    <collision>
+        <origin xyz="0.0 -0.01 -0.02" rpy="0.0 ${pi/2.0} 0.0"/>
         <geometry>
             <box size="0.1 0.012 0.035" />
@@ -245,16 +316,16 @@
 <link name="l_shoulder">
     <inertial>
-        <origin xyz="-0.016 0.044 0.0" rpy="-1.57 1.57 0.0"/>
+        <origin xyz="-0.016 -0.036 0.0" rpy="${-pi/2.0} ${pi/2.0} 0.0"/>
         <mass value="0.053"/>
         <inertia ixx="3.308e-4" ixy="9.972e-8" ixz="-2.037e-9" iyy="4.650e-5" iyz="2.113e-6" izz="3.545e-5"/>
     </inertial>
     <visual name="">
-        <origin xyz="0.0 -0.04 0.0" rpy="-1.57 1.57 0.0"/>
-        <geometry>
-            <mesh filename="package://reachy_description/meshes/shoulder.dae"/>
-        </geometry>
-    </visual>
-    <collision>
-        <origin xyz="0.0 -0.04 0.0" rpy="-1.57 1.57 0.0"/>
+        <origin xyz="0.0 -0.04 0.0" rpy="${-pi/2.0} ${pi/2.0} 0.0"/>
+        <geometry>
+            <mesh filename="file://$(find reachy_description)/meshes/shoulder.dae"/>
+        </geometry>
+    </visual>
+    <collision>
+        <origin xyz="0.0 -0.04 0.0" rpy="${-pi/2.0} ${pi/2.0} 0.0"/>
         <geometry>
             <cylinder length="0.09" radius="0.035" />
@@ -266,10 +337,10 @@
         <origin xyz="0.0 0.0 -0.019" rpy="0.0 0.0 0.0"/>
         <mass value="0.158"/>
-        <inertia ixx="6.887e+4" ixy="5.393e+0" ixz="-9.155e+2" iyy="7.895e+4" iyz="4.512e-1" izz="4.235e+4"/>
-    </inertial>
-    <visual name="">
-        <origin xyz="0.0 0.0 0.0" rpy="0.0 0.0 0.0"/>
-        <geometry>
-            <mesh filename="package://reachy_description/meshes/shoulder_x.dae"/>
+        <inertia ixx="6.887e-5" ixy="5.393e-9" ixz="-9.155e-7" iyy="7.895e-5" iyz="4.512e-10" izz="4.235e-5"/>
+    </inertial>
+    <visual name="">
+        <origin xyz="0.0 0.0 0.0" rpy="0.0 0.0 0.0"/>
+        <geometry>
+            <mesh filename="file://$(find reachy_description)/meshes/shoulder_x.dae"/>
         </geometry>
     </visual>
@@ -290,5 +361,5 @@
         <origin xyz="0.0 0.0 -0.0526" rpy="0.0 0.0 0.0"/>
         <geometry>
-            <mesh filename="package://reachy_description/meshes/upper_arm.dae"/>
+            <mesh filename="file://$(find reachy_description)/meshes/upper_arm.dae"/>
         </geometry>
     </visual>
@@ -309,5 +380,5 @@
         <origin xyz="0.0 0.0 0.0" rpy="0.0 0.0 0.0"/>
         <geometry>
-            <mesh filename="package://reachy_description/meshes/forearm.dae"/>
+            <mesh filename="file://$(find reachy_description)/meshes/forearm.dae"/>
         </geometry>
     </visual>
@@ -328,5 +399,5 @@
         <origin xyz="0.0 0.0 -0.1" rpy="0.0 0.0 0.0"/>
         <geometry>
-            <mesh filename="package://reachy_description/meshes/wrist.dae"/>
+            <mesh filename="file://$(find reachy_description)/meshes/wrist.dae"/>
         </geometry>
     </visual>
@@ -347,5 +418,5 @@
         <origin xyz="0.0 0.0 0.0" rpy="0.0 0.0 0.0"/>
         <geometry>
-            <mesh filename="package://reachy_description/meshes/wrist2hand.dae"/>
+            <mesh filename="file://$(find reachy_description)/meshes/wrist2hand.dae"/>
         </geometry>
     </visual>
@@ -359,16 +430,18 @@
 <link name="l_gripper_thumb">
     <inertial>
-        <origin xyz="0.032 0.008 0.0" rpy="0.0 1.57 0.0"/>
+        <!-- <origin xyz="0.032 0.008 0.0" rpy="0.0 1.57 0.0"/> -->
+        <origin xyz="0.0 0.008 0.0" rpy="0.0 ${pi/2.0} 0.0"/>
         <mass value="0.173"/>
-        <inertia ixx="1.088e+5" ixy="3.479e+4" ixz="1.357e+3" iyy="1.422e+5" iyz="-7.930e+2" izz="2.116e+5"/>
-    </inertial>
-    <visual name="">
-        <origin xyz="0.0 0.0 0.0" rpy="0.0 1.57 0.0"/>
-        <geometry>
-            <mesh filename="package://reachy_description/meshes/l_gripper_thumb.dae"/>
-        </geometry>
-    </visual>
-    <collision>
-        <origin xyz="0.0 -0.02 -0.06" rpy="0.0 1.57 0.0"/>
+        <!-- <inertia ixx="1.088e+5" ixy="3.479e+4" ixz="1.357e+3" iyy="1.422e+5" iyz="-7.930e+2" izz="2.116e+5"/> -->
+        <inertia ixx="0.0001" izz="0.0001" iyy="0.0001" ixy="0" ixz="0" iyz="0" />
+    </inertial>
+    <visual name="">
+        <origin xyz="0.0 0.0 0.0" rpy="0.0 ${pi/2.0} 0.0"/>
+        <geometry>
+            <mesh filename="file://$(find reachy_description)/meshes/l_gripper_thumb.dae"/>
+        </geometry>
+    </visual>
+    <collision>
+        <origin xyz="0.0 -0.02 -0.06" rpy="0.0 ${pi/2.0} 0.0"/>
         <geometry>
             <box size="0.1 0.012 0.035" />
@@ -378,16 +451,18 @@
 <link name="l_gripper_finger">
     <inertial>
-        <origin xyz="0.005 -0.043 0.0" rpy="0.0 1.57 0.0"/>
+        <!-- <origin xyz="0.005 -0.043 0.0" rpy="0.0 1.57 0.0"/> -->
+        <origin xyz="-0.00 0.005 -0.0" rpy="${pi/2.0} 0.0 ${pi/2.0}"/>
         <mass value="0.035"/>
-        <inertia ixx="9.165e-5" ixy="6.559e-6" ixz="3.609e-10" iyy="1.062e-5" iyz="4.666e-9" izz="8.705e-5"/>
-    </inertial>
-    <visual name="">
-        <origin xyz="0.0 0.0 0.0" rpy="0.0 1.57 0.0"/>
-        <geometry>
-            <mesh filename="package://reachy_description/meshes/l_gripper_finger.dae"/>
-        </geometry>
-    </visual>
-    <collision>
-        <origin xyz="0.0 0.01 -0.02" rpy="0.0 1.57 0.0"/>
+        <!-- <inertia ixx="9.165e-5" ixy="6.559e-6" ixz="3.609e-10" iyy="1.062e-5" iyz="4.666e-9" izz="8.705e-5"/> -->
+        <inertia ixx="0.00005" izz="0.00005" iyy="0.00005" ixy="0" ixz="0" iyz="0" />
+    </inertial>
+    <visual name="">
+        <origin xyz="0.0 0.0 0.0" rpy="0.0 ${pi/2.0} 0.0"/>
+        <geometry>
+            <mesh filename="file://$(find reachy_description)/meshes/l_gripper_finger.dae"/>
+        </geometry>
+    </visual>
+    <collision>
+        <origin xyz="0.0 0.01 -0.02" rpy="0.0 ${pi/2.0} 0.0"/>
         <geometry>
             <box size="0.1 0.012 0.035" />
@@ -397,6 +472,11 @@
 <link name="left_tip"/>
 </xacro:if>
+<link name="world" />
+<joint name="world_to_pedestal=" type="fixed">
+     <parent link="world"/>
+     <child link="pedestal"/>
+</joint>
 <!-- Head and Torso joints -->
-<joint name="pedestal" type="fixed">
+<joint name="pedestal_link" type="fixed">
     <origin xyz="0 0 1" rpy="0 0 0" />
     <parent link="pedestal" />
@@ -407,14 +487,16 @@
     <origin xyz="-0.052 -0.057 0.086" rpy="-0.166 -1.054 1.11"/>
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